Commit message: Add files via upload

File: totem.urdf (robot description, URDF)
Before this commit: robot physics, 4 links, 3 joints
Links:
- removed link duck_stuff
- added link pizza_stuff, mass .001; collision mesh filename=pizza.obj scale=.05 .05 .05; visual mesh filename=pizza.obj scale=.05 .05 .05
Joints:
- joint jfixed_stuff: child duck_stuff -> pizza_stuff

File: totemwine.urdf (robot description, URDF)
Before this commit: robot physics, 4 links, 3 joints
Links:
- link wine_stuff: geometry collision mesh filename=glass.obj scale=.01 .01 .01; visual mesh filename=glass.obj scale=.01 .01 .01
Joints:
- joint jfixed_stuff: origin xyz=0 0 0.01 rpy=0 0 0 -> xyz=0 0 0 rpy=0 0 0

Commit message: Add files via upload
Last update for a while

File: totem.urdf (robot description, URDF)
Before this commit: robot physics, 4 links, 3 joints
Links:
- link pizza_stuff: geometry collision mesh filename=pizzatexturée4.obj scale=.05 .05 .05; visual mesh filename=pizzatexturée4.obj scale=.05 .05 .05

File: totempomme.urdf (robot description, URDF)
Before this commit: robot physics, 4 links, 3 joints
Links:
- link apple_stuff: geometry collision mesh filename=banana.obj scale=.03 .03 .03; visual mesh filename=banana.obj scale=.03 .03 .03

File: totemwine.urdf (robot description, URDF)
Before this commit: robot physics, 4 links, 3 joints
Links:
- link wine_stuff: geometry collision mesh filename=Wine_Bottle_White.obj scale=1 1 1; visual mesh filename=Wine_Bottle_White.obj scale=1 1 1
